File: hardware/logicboard/mkr1000_backpack.sch (EAGLE design)
At the start: 15 parts, among them J3 3.3V, J4 DNP, J5 DNP

Commit message: Fixed position of pinheader.
Parts:
- removed J1, J2: (no value), SparkFun-Connectors:CONN_02-JST-2-PTH-NO_SILK
- added LED1, LED2: (no value), SparkFun-Connectors:CONN_02-JST-2-PTH-NO_SILK
- renumbered J3 to I2C
Connections:
- removed net N$1: J1.1, R1.1
- removed net N$2: J2.1, R2.1
- removed net N$3: J1.2, J4.13
- removed net N$4: J2.2, J4.14
- new net LED1A: LED1.1, R1.1
- new net LED1K: J4.13, LED1.2
- new net LED2A: LED2.1, R2.1
- new net LED2K: J4.14, LED2.2
Changed lines of the file:
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@@
 <part name="C1" library="resistor" library_urn="urn:adsk.eagle:library:348" deviceset="C-US" device="025-025X050" package3d_urn="urn:adsk.eagle:package:26151/1" value="0.1u"/>
 <part name="ANALOG" library="con-ml" library_urn="urn:adsk.eagle:library:164" deviceset="ML14L" device="" package3d_urn="urn:adsk.eagle:package:8677/1"/>
-<part name="J1" library="SparkFun-Connectors" library_urn="urn:adsk.eagle:library:513" deviceset="CONN_02" device="-JST-2-PTH-NO_SILK" package3d_urn="urn:adsk.eagle:package:38056/1"/>
-<part name="J2" library="SparkFun-Connectors" library_urn="urn:adsk.eagle:library:513" deviceset="CONN_02" device="-JST-2-PTH-NO_SILK" package3d_urn="urn:adsk.eagle:package:38056/1"/>
-<part name="J3" library="SparkFun-Connectors" library_urn="urn:adsk.eagle:library:513" deviceset="CONN_05" device="SMD" package3d_urn="urn:adsk.eagle:package:38026/1" value="3.3V"/>
+<part name="LED1" library="SparkFun-Connectors" library_urn="urn:adsk.eagle:library:513" deviceset="CONN_02" device="-JST-2-PTH-NO_SILK" package3d_urn="urn:adsk.eagle:package:38056/1"/>
+<part name="LED2" library="SparkFun-Connectors" library_urn="urn:adsk.eagle:library:513" deviceset="CONN_02" device="-JST-2-PTH-NO_SILK" package3d_urn="urn:adsk.eagle:package:38056/1"/>
+<part name="I2C" library="SparkFun-Connectors" library_urn="urn:adsk.eagle:library:513" deviceset="CONN_05" device="SMD" package3d_urn="urn:adsk.eagle:package:38026/1" value="3.3V"/>
 <part name="SUPPLY3" library="supply2" library_urn="urn:adsk.eagle:library:372" deviceset="GND" device=""/>
 <part name="SUPPLY4" library="supply2" library_urn="urn:adsk.eagle:library:372" deviceset="GND" device=""/>
@@
 <instance part="C1" gate="G$1" x="320.04" y="121.92"/>
 <instance part="ANALOG" gate="1" x="279.4" y="149.86" rot="MR180"/>
-<instance part="J1" gate="G$1" x="340.36" y="111.76" rot="R180"/>
-<instance part="J2" gate="G$1" x="340.36" y="96.52" rot="R180"/>
-<instance part="J3" gate="G$1" x="375.92" y="81.28" rot="R180"/>
+<instance part="LED1" gate="G$1" x="342.9" y="111.76" rot="R180"/>
+<instance part="LED2" gate="G$1" x="342.9" y="96.52" rot="R180"/>
+<instance part="I2C" gate="G$1" x="375.92" y="81.28" rot="R180"/>
 <instance part="SUPPLY3" gate="GND" x="363.22" y="71.12"/>
 <instance part="SUPPLY4" gate="GND" x="365.76" y="93.98"/>
@@
 </segment>
 <segment>
-<pinref part="J3" gate="G$1" pin="5"/>
+<pinref part="I2C" gate="G$1" pin="5"/>
 <wire x1="368.3" y1="76.2" x2="363.22" y2="76.2" width="0.1524" layer="91"/>
 <pinref part="SUPPLY3" gate="GND" pin="GND"/>
@@
 <junction x="289.56" y="142.24"/>
 <wire x1="320.04" y1="127" x2="325.12" y2="127" width="0.1524" layer="91"/>
-<pinref part="J3" gate="G$1" pin="1"/>
+<pinref part="I2C" gate="G$1" pin="1"/>
 <wire x1="325.12" y1="127" x2="327.66" y2="127" width="0.1524" layer="91"/>
 <wire x1="327.66" y1="127" x2="358.14" y2="127" width="0.1524" layer="91"/>
@@
 </segment>
 </net>
-<net name="N$3" class="0">
+<net name="LED1K" class="0">
 <segment>
 <pinref part="J4" gate="G$1" pin="13"/>
@@
 <wire x1="271.78" y1="101.6" x2="271.78" y2="91.44" width="0.1524" layer="91"/>
 <wire x1="271.78" y1="91.44" x2="330.2" y2="91.44" width="0.1524" layer="91"/>
-<pinref part="J1" gate="G$1" pin="2"/>
+<pinref part="LED1" gate="G$1" pin="2"/>
 <wire x1="330.2" y1="91.44" x2="330.2" y2="109.22" width="0.1524" layer="91"/>
-<wire x1="330.2" y1="109.22" x2="332.74" y2="109.22" width="0.1524" layer="91"/>
-</segment>
-</net>
-<net name="N$4" class="0">
-<segment>
-<pinref part="J2" gate="G$1" pin="2"/>
+<wire x1="330.2" y1="109.22" x2="335.28" y2="109.22" width="0.1524" layer="91"/>
+</segment>
+</net>
+<net name="LED2K" class="0">
+<segment>
+<pinref part="LED2" gate="G$1" pin="2"/>
+<wire x1="335.28" y1="93.98" x2="332.74" y2="93.98" width="0.1524" layer="91"/>
 <wire x1="332.74" y1="93.98" x2="332.74" y2="88.9" width="0.1524" layer="91"/>
 <wire x1="332.74" y1="88.9" x2="330.2" y2="88.9" width="0.1524" layer="91"/>
@@
 <wire x1="309.88" y1="101.6" x2="309.88" y2="86.36" width="0.1524" layer="91"/>
 <wire x1="309.88" y1="86.36" x2="309.88" y2="83.82" width="0.1524" layer="91"/>
-<pinref part="J3" gate="G$1" pin="2"/>
+<pinref part="I2C" gate="G$1" pin="2"/>
 <wire x1="309.88" y1="83.82" x2="355.6" y2="83.82" width="0.1524" layer="91"/>
 <label x="363.22" y="83.82" size="1.778" layer="95"/>
@@
 <wire x1="304.8" y1="114.3" x2="312.42" y2="114.3" width="0.1524" layer="91"/>
 <wire x1="312.42" y1="114.3" x2="312.42" y2="81.28" width="0.1524" layer="91"/>
-<pinref part="J3" gate="G$1" pin="3"/>
+<pinref part="I2C" gate="G$1" pin="3"/>
 <wire x1="312.42" y1="81.28" x2="360.68" y2="81.28" width="0.1524" layer="91"/>
 <label x="363.22" y="81.28" size="1.778" layer="95"/>
@@
 <wire x1="304.8" y1="116.84" x2="314.96" y2="116.84" width="0.1524" layer="91"/>
 <wire x1="314.96" y1="116.84" x2="314.96" y2="78.74" width="0.1524" layer="91"/>
-<pinref part="J3" gate="G$1" pin="4"/>
+<pinref part="I2C" gate="G$1" pin="4"/>
 <wire x1="314.96" y1="78.74" x2="358.14" y2="78.74" width="0.1524" layer="91"/>
 <label x="363.22" y="78.74" size="1.778" layer="95"/>
@@
 </segment>
 </net>
-<net name="N$1" class="0">
+<net name="LED1A" class="0">
 <segment>
 <pinref part="R1" gate="G$1" pin="1"/>
 <wire x1="325.12" y1="114.3" x2="325.12" y2="111.76" width="0.1524" layer="91"/>
-<pinref part="J1" gate="G$1" pin="1"/>
-<wire x1="325.12" y1="111.76" x2="332.74" y2="111.76" width="0.1524" layer="91"/>
-</segment>
-</net>
-<net name="N$2" class="0">
+<pinref part="LED1" gate="G$1" pin="1"/>
+<wire x1="325.12" y1="111.76" x2="335.28" y2="111.76" width="0.1524" layer="91"/>
+</segment>
+</net>
+<net name="LED2A" class="0">
 <segment>
 <pinref part="R2" gate="G$1" pin="1"/>
 <wire x1="327.66" y1="99.06" x2="327.66" y2="96.52" width="0.1524" layer="91"/>
-<pinref part="J2" gate="G$1" pin="1"/>
-<wire x1="327.66" y1="96.52" x2="332.74" y2="96.52" width="0.1524" layer="91"/>
-</segment>
-</net>
+<pinref part="LED2" gate="G$1" pin="1"/>
+<wire x1="327.66" y1="96.52" x2="335.28" y2="96.52" width="0.1524" layer="91"/>
+</segment>
+</net>
