File: hardware/logicboard/pc1000-001.sch (EAGLE design)
At the start: 15 parts, among them J4 DNP, J5 DNP

Commit message: Name change.
Other:
- note added: "PineappleCake 1000 1.0.0"
- moved on the sheet: ANALOG, C1, I2C, IPADDRESS, J4, J5, LED1, LED2, MMA8452Q, R1, R2, R3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
